File: Schaltungen/prototyp_platine/prototyp_platine.kicad_pcb (KiCad board)
At the start: 2 copper layers, 0 parts

Commit message: Platinenentwurf fertig.
Parts:
- added C1: 10p, C1, F.Cu at (43.2, 141.0)
- added C2: 10p, C1, F.Cu at (41.9, 132.1)
- added C3: 10p, C1, F.Cu at (61.0, 141.0)
- added C4: 10p, C1, F.Cu at (54.6, 132.1)
- added C_K1: 10p, C1, F.Cu at (29.2, 129.5)
- added C_K2: 10p, C1, F.Cu at (47.0, 134.6)
- added C_K3: 1n, C1, F.Cu at (67.3, 129.5)
- added C_K4: >500p, 100n, C1, F.Cu at (81.3, 135.9)
- added C_S1: 100n, C1, F.Cu at (58.4, 156.2)
- added C_S2: 100n, C1, F.Cu at (43.2, 151.1)
- added D1: Grün (2,2V), LED-3MM, F.Cu at (54.6, 165.1)
- added D2: Gelb (2,1V), LED-3MM, F.Cu at (54.6, 160.0)
- added D3: Rot (2V), LED-3MM, F.Cu at (54.6, 154.9)
- added P1: CONN_5X2, VASCH5x2, F.Cu at (71.1, 161.3)
- added Q1: BC337, TO92-EBC, F.Cu at (77.5, 146.1)
- added R1: 100k, RV2, F.Cu at (24.1, 132.1)
- added R10: 560k, R3, F.Cu at (58.4, 143.5)
- added R11: 4k, R3, F.Cu at (73.7, 133.3)
- added R12: 100k, RV2, F.Cu at (77.5, 134.6)
- added R13: 10k, R1, F.Cu at (80.0, 149.9)
- added R14: 1,5k, R1, F.Cu at (49.5, 165.1)
- added R15: 1,5k, R3, F.Cu at (47.0, 162.6)
- added R16: 1,5k, R1, F.Cu at (49.5, 154.9)
- added R17: 10k, R4, F.Cu at (76.2, 167.6)
- added R18: 10k, R3, F.Cu at (77.5, 182.9)
- added R19: 10k, R1, F.Cu at (78.7, 180.3)
- added R2: 10k, R3, F.Cu at (25.4, 143.5)
- added R3: 390k, R3, F.Cu at (36.8, 129.5)
- added R4: 390k, R3, F.Cu at (38.1, 135.9)
- added R5: 330k, R1, F.Cu at (43.2, 135.9)
- added R6: 560k, R4, F.Cu at (40.6, 142.2)
- added R7: 390k, R1, F.Cu at (52.1, 134.6)
- added R8: 390k, R3, F.Cu at (57.1, 137.2)
- added R9: 330k, R1, F.Cu at (61.0, 133.3)
- added R_B1: 1k, R3, F.Cu at (39.4, 157.5)
- added R_B2: 1k, R3, F.Cu at (31.8, 162.6)
- added R_U1: 47k, R1, F.Cu at (81.3, 146.1)
- added R_U2: 10k, RV2, F.Cu at (76.2, 141.0)
- added Rec1: Empfänger, PIN_ARRAY_3X1, F.Cu at (17.8, 139.7)
- added SW1: SW_PUSH, SW_PUSH_SMALL, F.Cu at (67.3, 172.7)
- added Send1: 2,55n, PIN_ARRAY_3X1, F.Cu at (17.8, 154.9)
- added T1: BC337, TO92-EBC, F.Cu at (31.8, 156.2)
- added T2: BC327, TO92-EBC, F.Cu at (26.7, 156.2)
- added U1: LM358N, DIP-8__300, F.Cu at (31.8, 135.9)
- added U2: LM358N, DIP-8__300, F.Cu at (67.3, 135.9)
- added Z1: 4V, D3, F.Cu at (36.8, 152.4)
- added Z2: 12V, D3, F.Cu at (39.4, 160.0)
- added µC1: ATMEGA8-P, DIP-28__300, F.Cu at (36.8, 176.5)
Routing:
- net GND: track 0.00 -> 205.7 mm, vias 0 -> 6
- net +5V: track 0.00 -> 105.4 mm, vias 0 -> 2
- net +12V: track 0.00 -> 102.7 mm, vias 0 -> 5
- net -12V: track 0.00 -> 100.9 mm, vias 0 -> 5
- net /Empfänger/Signal: track 0.00 -> 72.9 mm, vias 0 -> 2
- net MISO: track 0.00 -> 66.0 mm, vias 0 -> 2
- net SCK: track 0.00 -> 66.0 mm, vias 0 -> 2
- net MOSI: track 0.00 -> 62.3 mm, vias 0 -> 4
- net N-0000019: track 0.00 -> 51.9 mm, vias 0 -> 1
- net SDA: track 0.00 -> 45.7 mm
- net SCL: track 0.00 -> 41.9 mm, vias 0 -> 2
- net /Mikrocontroller/40kHz PWM: track 0.00 -> 41.3 mm, vias 0 -> 1
- net N-0000021: track 0.00 -> 29.0 mm, vias 0 -> 1
- net Reset: track 0.00 -> 20.3 mm, vias 0 -> 2
- net N-0000048: track 0.00 -> 14.8 mm, vias 0 -> 1
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