File: Schaltungen/prototyp_platine_v2/prototyp_platine.kicad_pcb (KiCad board)
At the start: 2 copper layers, 47 parts, among them P1 CONN_5X2, Q1 BC337, SW1 SW_PUSH, T1 BC337, T2 BC327, T3 BC337, T4 BC327, U1 LM358N, U2 LM358N

Commit message: Prototyp-Platine..
Parts:
- R18, R19: footprint R3 -> R4
- moved D2 35.9 mm to (87.6, 167.6), turned to 180 degrees
- moved D1 34.9 mm to (87.6, 165.1), turned to 180 degrees
- moved R20 17.6 mm to (100.3, 149.9), turned to 0 degrees
- moved D3 15.3 mm to (87.6, 170.2), turned to 180 degrees
- moved SW1 13.7 mm to (108.0, 149.9), turned to 0 degrees
- moved R17 8.13 mm to (95.2, 165.1), turned to 180 degrees
- moved R19 8.03 mm to (96.5, 170.2), turned to 0 degrees
- moved R18 5.68 mm to (86.4, 167.6)
- moved R10 3.59 mm to (76.2, 144.8), turned to 90 degrees
- moved C_S1 2.84 mm to (95.2, 152.4)
- moved µC1 2.84 mm to (95.2, 158.8)
Routing:
- net GND: track 129.5 -> 204.3 mm, vias 2 -> 4
- net +5V: track 27.9 -> 101.6 mm, vias 2 -> 4
- net MOSI: track 15.2 -> 44.4 mm, vias 0 -> 2
- net SCK: track 0.00 -> 27.2 mm
- net MISO: track 0.00 -> 22.9 mm
- net /Mikrocontroller/Empfänger/Signal: track 0.00 -> 8.67 mm
- net N-0000022: track 0.00 -> 7.62 mm
- net Reset: track 0.00 -> 5.08 mm
- net /Mikrocontroller/Sender/40kHz PWM: track 0.00 -> 5.08 mm
- net N-0000032: track 0.00 -> 2.54 mm
- net N-0000024: track 0.00 -> 2.54 mm
- net N-0000017: track 0.00 -> 2.54 mm
- net N-0000016: track 0.00 -> 2.54 mm

Commit message: Schema fertig.
Parts:
- R10, R15: footprint R4 -> R3
- R11: footprint R4 -> R5
- R20: footprint R3 -> R6
- RB2: footprint R1 -> R3
- moved SW1 20.5 mm to (110.5, 170.2), turned to 180 degrees
- moved RB2 6.48 mm to (54.6, 167.6), turned to 180 degrees
- moved R20 3.81 mm to (104.1, 149.9)
- moved R10 2.84 mm to (78.7, 146.1)
- moved R12 2.54 mm to (35.6, 161.3)
- moved C4 2.54 mm to (26.7, 154.9)
- moved T1 2.54 mm to (26.7, 158.8)
- moved R13 2.54 mm to (30.5, 153.7)
- moved R14 2.54 mm to (31.8, 162.6)
- moved R16 2.54 mm to (45.7, 161.3)
- moved T2 2.54 mm to (34.3, 158.8)
- moved T3 2.54 mm to (41.9, 163.8)
- moved T4 2.54 mm to (49.5, 163.8)
- moved R15 1.27 mm to (54.6, 160.0)
- moved R11 1.27 mm to (22.9, 153.7)
Routing:
- net Reset: track 5.08 -> 76.2 mm, vias 0 -> 2
- net /Mikrocontroller/Empfänger/Signal: track 8.67 -> 46.6 mm
- net GND: track 204.3 -> 233.7 mm
- net /Mikrocontroller/Sender/40kHz PWM: track 5.08 -> 27.9 mm, vias 0 -> 2
- net +5V: track 101.6 -> 120.6 mm
- net N-0000047: track 5.08 -> 12.7 mm
- net +12V: track 82.3 -> 84.9 mm
- net -12V: track 68.6 -> 71.1 mm
- net N-0000035: track 5.08 -> 7.62 mm
- net N-0000040: track 3.59 -> 6.13 mm, vias 0 -> 1
- net MOSI: track 44.4 -> 45.7 mm
