File: Schaltungen/prototyp_platine_v2/prototyp_platine.kicad_pcb (KiCad board)
At the start: 2 copper layers, 47 parts, among them P1 CONN_5X2, Q1 BC337, SW1 SW_PUSH, T1 BC337, T2 BC327, T3 BC337, T4 BC327, U1 LM358N, U2 LM358N

Commit message: Update von Firmware und Schaltungen.
Parts:
- moved T1 5.68 mm to (24.1, 163.8), turned to 270 degrees
Connections:
- RV2 pad 2: (no net) -> N-0000045
- T1 pad C: N-0000033 -> N-0000036
- T1 pad E: N-0000036 -> N-0000033
- U2 pad 1: (no net) -> N-0000044
- U2 pad 2: (no net) -> N-0000045
- U2 pad 3: (no net) -> N-0000043
Routing:
- net N-0000045: track 0.00 -> 4.34 mm
- net (no net): track 4.34 -> 0.00 mm
- net N-0000039: track 7.62 -> 10.2 mm
